File: hardware/KiCad/ESC_v1.0/_autosave-ESC_v1.0.kicad_pcb (KiCad board)
At the start: 2 copper layers, 68 parts, among them J3 Conn_ARM_SWD_TagConnect_TC203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, Q1 NVMFS5C604N, Q2 NVMFS5C604N, U1 STM32G484CEU6, U2 LM5160A, U3 TPS7B92033, U4 2EDL8024, U5 USBLC6-2SC6, X1 16MHz

Commit message: Update kicad and docs
Parts:
- added C18: 1u, Capacitor_SMD:C_0603_1608Metric, F.Cu at (127.1, 81.3)
- added C20: 1u, Capacitor_SMD:C_0603_1608Metric, F.Cu at (127.1, 83.8)
- added C21: 100p, Capacitor_SMD:C_0805_2012Metric, F.Cu at (139.3, 81.5)
- added C22: 100p, Capacitor_SMD:C_0805_2012Metric, F.Cu at (139.3, 84.5)
- added C23: 100p, Capacitor_SMD:C_0805_2012Metric, F.Cu at (139.3, 87.5)
- added C24: 100n, Capacitor_SMD:C_0402_1005Metric, F.Cu at (138.5, 95.2)
- added C26: 1u, Capacitor_SMD:C_0603_1608Metric, F.Cu at (185.4, 77.4)
- added C27: 1u, Capacitor_SMD:C_0603_1608Metric, F.Cu at (185.4, 79.9)
- added C28: 100n, Capacitor_SMD:C_0402_1005Metric, F.Cu at (188.9, 91.9)
- added C30: 100n, Capacitor_SMD:C_0402_1005Metric, F.Cu at (188.9, 93.8)
- added C31: 100n, Capacitor_SMD:C_0402_1005Metric, F.Cu at (188.9, 95.8)
- added C34: 1u, Capacitor_SMD:C_0603_1608Metric, F.Cu at (185.4, 82.4)
- added C35: 1u, Capacitor_SMD:C_0603_1608Metric, F.Cu at (185.4, 84.9)
- added C39: 100n, Capacitor_SMD:C_0402_1005Metric, F.Cu at (188.9, 97.8)
- added C40: 100n, Capacitor_SMD:C_0402_1005Metric, F.Cu at (188.9, 99.8)
- added C41: 100n, Capacitor_SMD:C_0402_1005Metric, F.Cu at (188.9, 101.7)
- added D2: KT-0603W, LED_SMD:LED_0603_1608Metric, F.Cu at (139.1, 90.3)
- added D3: KT-0603W, LED_SMD:LED_0603_1608Metric, F.Cu at (139.1, 92.9)
- added Q3: NVMFS5C604N, Package_SO:ONSemi_SO-8FL_488AA, F.Cu at (179.4, 79.7)
- added Q4: NVMFS5C604N, Package_SO:ONSemi_SO-8FL_488AA, F.Cu at (179.4, 86.8)
- added Q5: NVMFS5C604N, Package_SO:ONSemi_SO-8FL_488AA, F.Cu at (179.4, 93.9)
- added Q6: NVMFS5C604N, Package_SO:ONSemi_SO-8FL_488AA, F.Cu at (179.4, 101.0)
- added R1: 5.1, Resistor_SMD:R_0805_2012Metric, F.Cu at (189.6, 77.6)
- added R10: 47, Resistor_SMD:R_0603_1608Metric, F.Cu at (131.1, 88.8)
- added R12: 47, Resistor_SMD:R_0603_1608Metric, F.Cu at (131.1, 91.3)
- added R13: 390, Resistor_SMD:R_0603_1608Metric, F.Cu at (131.1, 93.8)
- added R14: 390, Resistor_SMD:R_0603_1608Metric, F.Cu at (131.1, 96.3)
- added R15: 5.6k, Resistor_SMD:R_0603_1608Metric, F.Cu at (135.1, 81.3)
- added R16: 150, Resistor_SMD:R_0603_1608Metric, F.Cu at (135.1, 83.8)
- added R17: 150, Resistor_SMD:R_0603_1608Metric, F.Cu at (135.1, 86.3)
- added R18: 150, Resistor_SMD:R_0603_1608Metric, F.Cu at (135.1, 88.8)
- added R2: 390, Resistor_SMD:R_0603_1608Metric, F.Cu at (127.1, 86.3)
- added R20: 39k, Resistor_SMD:R_0603_1608Metric, F.Cu at (135.1, 91.3)
- added R21: 1k, Resistor_SMD:R_0603_1608Metric, F.Cu at (135.1, 93.8)
- added R22: 120k, Resistor_SMD:R_0603_1608Metric, F.Cu at (135.1, 96.3)
- added R23: 10, Resistor_SMD:R_0805_2012Metric, F.Cu at (189.6, 80.6)
- added R24: 10, Resistor_SMD:R_0805_2012Metric, F.Cu at (189.6, 83.5)
- added R25: 10, Resistor_SMD:R_0805_2012Metric, F.Cu at (189.6, 86.5)
- added R26: 10, Resistor_SMD:R_0805_2012Metric, F.Cu at (189.6, 89.4)
- added R27: 10k, Resistor_SMD:R_0603_1608Metric, F.Cu at (185.4, 87.4)
- added R28: 10k, Resistor_SMD:R_0603_1608Metric, F.Cu at (185.4, 90.0)
- added R3: 22k, Resistor_SMD:R_0603_1608Metric, F.Cu at (127.1, 88.8)
- added R30: 0.5, ESC-FootprintLib:Kelvin Shunt 1216 (3038), F.Cu at (191.6, 91.7)
- added R31: 5.1, Resistor_SMD:R_0805_2012Metric, F.Cu at (194.1, 77.6)
- added R38: 10, Resistor_SMD:R_0805_2012Metric, F.Cu at (194.1, 80.6)
- added R39: 10, Resistor_SMD:R_0805_2012Metric, F.Cu at (194.1, 83.5)
- added R4: 200k, Resistor_SMD:R_0603_1608Metric, F.Cu at (127.1, 91.3)
- added R40: 10, Resistor_SMD:R_0805_2012Metric, F.Cu at (194.1, 86.5)
- added R41: 10, Resistor_SMD:R_0805_2012Metric, F.Cu at (194.1, 89.4)
- added R42: 10k, Resistor_SMD:R_0603_1608Metric, F.Cu at (185.4, 92.5)
- added R43: 10k, Resistor_SMD:R_0603_1608Metric, F.Cu at (185.4, 95.0)
- added R44: 0.5, ESC-FootprintLib:Kelvin Shunt 1216 (3038), F.Cu at (196.2, 91.7)
- added R5: 120k, Resistor_SMD:R_0603_1608Metric, F.Cu at (127.1, 93.8)
- added R6: 5.6k, Resistor_SMD:R_0603_1608Metric, F.Cu at (127.1, 96.3)
- added R7: 5.6k, Resistor_SMD:R_0603_1608Metric, F.Cu at (131.1, 81.3)
- added R8: 390, Resistor_SMD:R_0603_1608Metric, F.Cu at (131.1, 83.8)
- added R9: 47, Resistor_SMD:R_0603_1608Metric, F.Cu at (131.1, 86.3)
- added U5: 2EDL8024, Package_DFN_QFN:DFN-8-1EP_4x4mm_P0.8mm_EP2.5x3.6mm, F.Cu at (199.9, 79.0)
- added U6: 2EDL8024, Package_DFN_QFN:DFN-8-1EP_4x4mm_P0.8mm_EP2.5x3.6mm, F.Cu at (199.9, 84.8)
Connections:
- R19 pad 1: +10V -> Net-(U2-FB)
- R19 pad 2: Net-(U2-FB) -> AGND
