File: hardware/KiCad/ESC_v1.0/_autosave-ESC_v1.0.kicad_sch (KiCad schematic)
At the start: 105 parts, among them J1 Conn_01x03_Socket, J2 Conn_01x03_Socket, J3 Conn_ARM_SWD_TagConnect_TC203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, Q1 CSD18540Q5B, Q2 CSD18540Q5B, U1 STM32G484CEU6, U2 LM5160A, U3 TPS7B92033, U4 2EDL8024, X1 16MHz

Commit message: Final excel version
Parts:
- removed Cadc,ext, Csamp: 100n, Capacitor_SMD:C_0402_1005Metric, symbol ESC-SchemSymLib:CL05B104KO5NNNC
- removed Radc,ext, Radc,int, Rv1, Rv2: 10, Resistor_SMD:R_0805_2012Metric, symbol ESC-SchemSymLib:0805W8F100JT5E
Other:
- note removed: "MCU"
