File: hardware/KiCad/ESC_v1.0/ESC_v1.0.kicad_sch (KiCad schematic)
At the start: 159 parts, among them J1 Conn_01x03_Socket, J2 Conn_01x03_Socket, J3 Conn_ARM_SWD_TagConnect_TC203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, Q1 NVMFS5C604N, Q2 NVMFS5C604N, Q3 NVMFS5C604N, Q4 NVMFS5C604N, Q5 NVMFS5C604N, Q6 NVMFS5C604N, U1 STM32G484CEU6, U2 LM5160A, U3 TPS7B92033, U4 2EDL8024, U5 2EDL8024, U6 2EDL8024, X1 16MHz

Commit message: Kicad and esc choice review
Parts:
- removed C26, C27, C34, C35: 1u, Capacitor_SMD:C_0603_1608Metric, symbol ESC-SchemSymLib:CL10A105KB8NNNC
- removed C28, C30, C31, C39, C40, C41: 100n, Capacitor_SMD:C_0402_1005Metric, symbol ESC-SchemSymLib:CL05B104KO5NNNC
- removed D10, D11, D12, D4, D8, D9: RB161QS-40T18R, ESC-FootprintLib:Rohm_SMD1006, symbol ESC-SchemSymLib:RB161QS-40T18R
- removed Q1, Q2, Q3, Q4, Q5, Q6: NVMFS5C604N, ESC-FootprintLib:Onsemi_DFN5_DFNW5, symbol ESC-SchemSymLib:NVMFS5C604NL
- removed R1, R31: 5.1, Resistor_SMD:R_0805_2012Metric, symbol ESC-SchemSymLib:0805W8F510KT5E
- removed R23, R24, R25, R26, R38, R39, R40, R41: 10, Resistor_SMD:R_0805_2012Metric, symbol ESC-SchemSymLib:0805W8F100JT5E
- removed R27, R28, R42, R43: 10k, Resistor_SMD:R_0603_1608Metric, symbol ESC-SchemSymLib:0603WAF1002T5E
- removed R30, R44: 0.5, ESC-FootprintLib:Kelvin Shunt 1216 (3038), symbol ESC-SchemSymLib:HoBB1216-5W-0.5mR-1%
- removed TP16, TP27, TP28, TP29, TP30, TP31, TP32, TP33, TP34, TP35, TP36, TP37, TP38, TP39, TP40, TP41, TP42, TP43, TP44, TP6: TestPoint, symbol Connector:TestPoint
- removed U5, U6: 2EDL8024, Package_DFN_QFN:DFN-8-1EP_4x4mm_P0.8mm_EP2.5x3.6mm, symbol ESC-SchemSymLib:2EDL8024
- added Q1, Q2: CSD18540Q5B, ESC-FootprintLib:TRANS_CSD18540Q5B, symbol ESC-SchemSymLib:CSD18540Q5B
Connections:
- net ISENSE1: now also Q2.3 (S)
- net PH1: now also Q1.3 (S), Q2.1 (D)
- net VM: now also Q1.1 (D)
- net at R11.1, R34.2, R35.2: now also Q2.2 (G)
- net at R32.2, R33.2, R36.1: now also Q1.2 (G)

Commit message: Update kicad
Parts:
- removed C10, C11: 10p, Capacitor_SMD:C_0402_1005Metric, symbol ESC-SchemSymLib:CL05C100JB5NNNC
- removed C12, C13: 330u, symbol Device:C_Polarized
- removed C14, C15, C16, C17: 22u, Capacitor_SMD:C_0805_2012Metric, symbol ESC-SchemSymLib:CL21A475KAQNNNE
- removed C2, C3, C36, C37, C38: 100n, Capacitor_SMD:C_0402_1005Metric, symbol ESC-SchemSymLib:CL05B104KO5NNNC
- removed C32, C33: 1u, Capacitor_SMD:C_0603_1608Metric, symbol ESC-SchemSymLib:CL10A105KB8NNNC
- removed D1: D_TVS, symbol ESC-SchemSymLib:D_TVS
- removed J2: Conn_01x03_Socket, symbol Connector:Conn_01x03_Socket
- removed R10, R12, R9: 47, Resistor_SMD:R_0603_1608Metric, symbol ESC-SchemSymLib:0603WAF470JT5E
- removed R11, R19, R36: 10k, Resistor_SMD:R_0603_1608Metric, symbol ESC-SchemSymLib:0603WAF1002T5E
- removed R13, R14, R2, R8: 390, Resistor_SMD:R_0603_1608Metric, symbol ESC-SchemSymLib:0603WAF3900T5E
- removed R15, R6, R7: 5.6k, Resistor_SMD:R_0603_1608Metric, symbol ESC-SchemSymLib:0603WAF5601T5E
- removed R16, R17, R18: 150, Resistor_SMD:R_0603_1608Metric, symbol ESC-SchemSymLib:0603WAF1500T5E
- removed R20: 39k, Resistor_SMD:R_0603_1608Metric, symbol ESC-SchemSymLib:0603WAF3902T5E
- removed R21: 1k, Resistor_SMD:R_0603_1608Metric, symbol ESC-SchemSymLib:0603WAF1001T5E
- removed R22: 120k, Resistor_SMD:R_0603_1608Metric, symbol ESC-SchemSymLib:0603WAF1203T5E
- removed R29: 5.1, Resistor_SMD:R_0805_2012Metric, symbol ESC-SchemSymLib:0805W8F510KT5E
- removed R32, R33, R34, R35: 10, Resistor_SMD:R_0805_2012Metric, symbol ESC-SchemSymLib:0805W8F100JT5E
- removed R4: 200k, Resistor_SMD:R_0603_1608Metric, symbol ESC-SchemSymLib:0603WAF2003T5E
- removed TP1, TP10, TP11, TP12, TP13, TP14, TP15, TP17, TP18, TP19, TP2, TP20, TP21, TP22, TP23, TP24, TP25, TP26, TP3, TP4, TP7, TP8, TP9: TestPoint, symbol Connector:TestPoint
- removed TP5: ResetPad, symbol Connector:TestPoint
- removed X1: 16MHz, Crystal:Crystal_SMD_2520-4Pin_2.5x2.0mm, symbol ESC-SchemSymLib:Crystal_GND24
- added AP1: ActionPad, TestPoint:TestPoint_Pad_1.5x1.5mm, symbol ESC-SchemSymLib:ActionPad
- added C1, C2, C3, C4: 2.2u, Capacitor_SMD:C_1206_3216Metric, symbol ESC-SchemSymLib:CL31B225KBHNNNE
- added C16, C17: 100n, Capacitor_SMD:C_0402_1005Metric, symbol ESC-SchemSymLib:CL05B104KO5NNNC
- added C5: 1u, Capacitor_SMD:C_0603_1608Metric, symbol ESC-SchemSymLib:CL10A105KB8NNNC
- added C6: 220n, Capacitor_SMD:C_0402_1005Metric, symbol ESC-SchemSymLib:CL05B224KO5NNNC
- added PH1: ~, TestPoint:TestPoint_Pad_4.0x4.0mm, symbol ESC-SchemSymLib:PhaseConnector
- added R1, R3, R8: 3.3, Resistor_SMD:R_0402_1005Metric, symbol ESC-SchemSymLib:0402WGJ033JTCE
- added R10, R23, R25, R26: 1k, Resistor_SMD:R_0402_1005Metric, symbol ESC-SchemSymLib:0402WGF1001TCE
- added R11, R2: 10, Resistor_SMD:R_0402_1005Metric, symbol ESC-SchemSymLib:0402WGF100JTCE
- added R13, R16, R17, R30, R4: 10k, Resistor_SMD:R_0402_1005Metric, symbol ESC-SchemSymLib:0402WGF1002TCE
- added R14: 12k, Resistor_SMD:R_0402_1005Metric, symbol ESC-SchemSymLib:0402WGF1202TCE
- added R18, R19, R27, R28, R7: 100, Resistor_SMD:R_0402_1005Metric, symbol ESC-SchemSymLib:0402WGF1000TCE
- added R20, R6: 200k, Resistor_SMD:R_0402_1005Metric, symbol ESC-SchemSymLib:0402WGF2003TCE
- added R21, R22, R24: 33, Resistor_SMD:R_0402_1005Metric, symbol ESC-SchemSymLib:0402WGF330JTCE
- added R9: 51k, Resistor_SMD:R_0402_1005Metric, symbol ESC-SchemSymLib:0402WGF5102TCE
- C22: renamed from C23; footprint Capacitor_SMD:C_0805_2012Metric -> Capacitor_SMD:C_0603_1608Metric
- C23: renamed from C22; footprint Capacitor_SMD:C_0805_2012Metric -> Capacitor_SMD:C_0603_1608Metric
- C24: renamed from C21; footprint Capacitor_SMD:C_0805_2012Metric -> Capacitor_SMD:C_0603_1608Metric
- LED1: footprint FC-FootprintLib:SMD-B_19-337C_EVE -> ESC-FootprintLib:SMD-B_19-337C_EVE
- renumbered C29 to C10, C19 to C11, C20 to C12, C5 to C13, C6 to C14, C1 to C15, C4 to C18, C7 to C19, C9 to C20, C24 to C21, C8 to C25, C25 to C8, C18 to C9, D5 to D2, D6 to D3, D3 to D4, D7 to D5, D2 to D6, J3 to J1, J1 to J2, R3 to R12, R37 to R15, U4 to U1, U1 to U4
Connections:
- net +10V: now also C5.1, R8.1; no longer C9.1, L1.2, U3.1 (VIN)
- net +3V3: now also C16.1, C17.1, R7.1
- net AGND: now also C16.2, C17.2, C5.2, R13.2, R14.2, R20.2, R23.2, R25.2, R26.2
- net BOOT0: now also AP1.1, R20.1
- net HB1: now also C6.1
- net HO1: now also C6.2, R1.1
- net LED_B_K: now also R19.2
- net LED_G_K: now also R18.2
- net LED_R_K: now also R27.1
- net LO1: now also R3.1
- net PGND: now also C1.2, C2.2, C3.2, C4.2
- net PH1: now also PH1.1 (Pin_1), R16.2, R4.2
- net PH2: now also R17.2
- net PH3: now also R30.2
- net RGB_LED_B: now also R19.1
- net RGB_LED_G: now also R18.1
- net RGB_LED_R: now also R28.1
- net VM: now also C1.1, C2.1, C3.1, C4.1, R6.1
- net VSENSE1: now also C22.1, R24.2
- net VSENSE2: now also C23.1, R21.2
- net VSENSE3: now also C24.1, R22.2
- net at D6.2 (A): now also R10.2
- net at R12.1, U2.4 (EN/UVLO): now also R6.2
- net at D2.2 (A): now also R8.2
- net at U2.8 (FB): now also R14.1, R9.2
- net at D4.2 (A): now also R7.2
- net at Q1.2 (G): now also R1.2, R2.2, R4.1
- net at D5.2 (A): now also R11.1
- net at Q2.2 (G): now also R11.2, R13.1, R3.2
- net at D3.2 (A): now also R2.1
- net +10VNoise renamed +10.5VNoise
- new net: R17.1, R21.1, R23.1
- new net: R16.1, R22.1, R26.1
- new net: R27.2, R28.2
- new net: R24.1, R25.1, R30.1
- new net +10.5V: C9.1, L1.2, R10.1, R9.1, U3.1 (VIN)
Other:
- note added: "VM to 10.5V BUCK"
- note removed: "C_L1 = C_L2 = 2*(C_L - C_p) Assume stray capacitance C_p = 4pF R_EXT = 1/(2piFC_L2) !!!!!!!!!"
- note removed: "Crystal Oscillator"
- note removed: "General: Here we set OUT=(1A,10V), VIN=[4S, 6S]=[12, 60]V (ripple) --------------- Switching: FSW = min(FSW_max@VIN_min, FSW_max@VIN_max) = 981kHz RON = VOUT/FSW*10^10 = 110kR (TON=458ns) COT type BUCK: SW node high for TON if FB<REF. --------------- Inductor: L=VOx(VIN_max-VO)/(VIN_max*FSW*IO_max*0.4)=18µH. --------------- Other: Soft Start: CSS=1µF => TSS=200ms. Feedback: 10V to 2V => RFB2/RFB1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"
- note removed: "RGB LED TIM4 R = 65 : 296 (20mA : 5mA)"
- note removed: "VM to 10V BUCK"
- moved on the sheet: C13, C14, C15, C18, C22, C23, C24, D2, D3, D5, Q1, Q2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

Commit message: Kicad
Parts:
- added C26, C28, C7: 100p, Capacitor_SMD:C_0603_1608Metric, symbol ESC-SchemSymLib:CL10C101JB8NNNC
- added C27: 100n, Capacitor_SMD:C_0402_1005Metric, symbol ESC-SchemSymLib:CL05B104KO5NNNC
- added C43: 1u, Capacitor_SMD:C_0402_1005Metric, symbol FC-SchemSymbolLib:CL05A105KA5NQNC
- added C44: 100n, Capacitor_SMD:C_0402_1005Metric, symbol FC-SchemSymbolLib:CL05B104KO5NNNC
- added D1: ESD5Zxx, Diode_SMD:D_SOD-523, symbol Diode:ESD5Zxx
- added D7: LED, LED_SMD:LED_0603_1608Metric, symbol Device:LED
- added F1: Polyfuse, Resistor_SMD:R_1812_4532Metric, symbol Device:Polyfuse
- added J3: USB4105-GF-A, ESC-FootprintLib:GCT_USB4105-GF-A, symbol FC-SchemSymbolLib:USB4105-GF-A
- added NT1, NT3, NT4, NT5, NT6, NT7, NT8: NetTie_3_Tee, symbol Device:NetTie_3_Tee
- added NT2: NetTie_4_Cross, symbol Device:NetTie_4_Cross
- added R29, R39: 33, Resistor_SMD:R_0402_1005Metric, symbol ESC-SchemSymLib:0402WGF330JTCE
- added R31, R34, R35: 5.1k, Resistor_SMD:R_0402_1005Metric, symbol FC-SchemSymbolLib:0402WGF5101TCE
- added R32: 10k, Resistor_SMD:R_0402_1005Metric, symbol FC-SchemSymbolLib:0402WGF1002TCE
- added R33: 220, Resistor_SMD:R_0402_1005Metric, symbol FC-SchemSymbolLib:0402WGF2200TCE
- added R36, R40, R41: 10k, Resistor_SMD:R_0402_1005Metric, symbol ESC-SchemSymLib:0402WGF1002TCE
- added R37: 200k, Resistor_SMD:R_0402_1005Metric, symbol ESC-SchemSymLib:0402WGF2003TCE
- added R38: 1k, Resistor_SMD:R_0402_1005Metric, symbol ESC-SchemSymLib:0402WGF1001TCE
- added TH1: Thermistor_NTC, Resistor_SMD:R_0402_1005Metric, symbol ESC-SchemSymLib:NTCG103JF103FT1
- added TP4: TestPoint, TestPoint:TestPoint_Pad_D1.0mm, symbol Connector:TestPoint
- added U8: TPD2EUSB30A, Package_TO_SOT_SMD:Texas_DRT-3, symbol Power_Protection:TPD2EUSB30A
- D2, D3, D5: Manufacturer ROHM Semicon -> ROHM Semicon; Manufacturer Part Number RB161QS-40T18R -> RB161QS-40T18R; Supplier Link 1 (none) -> https://www.digikey.com.au/en/products/detail/rohm-semicond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; Supplier Link 2 (none) -> https://au.mouser.com/ProductDetail/ROHM-Semiconductor/RB16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
- R12: footprint Resistor_SMD:R_0603_1608Metric -> Resistor_SMD:R_0402_1005Metric
- R15: value 0.5 -> 0.5m
- U1: footprint Package_DFN_QFN:DFN-8-1EP_4x4mm_P0.8mm_EP2.5x3.6mm -> ESC-FootprintLib:2EDL8x2x_PG-VDSON-8-4
- U2: footprint Package_SON:WSON-12-1EP_4x4mm_P0.5mm_EP2.6x3mm_ThermalVias -> Package_SON:WSON-12-1EP_4x4mm_P0.5mm_EP2.6x3mm
Connections:
- net +3V3: now also R40.2
- net AGND: no longer C10.2, C11.2, C12.2, C15.2, C16.2, C17.2, C18.2, C21.2, C22.2, C23.2, C24.2, C25.2, C5.2, C9.2, D4.1 (K), D6.1 (K), J1.5 (GND), R12.2, R13.2, R14.2, R15.2, R20.2, R23.2, R25.2, R26.2, U1.7 (VSS), U1.PAD (VSS), U2.1 (AGND), U2.2 (PGND), U2.PAD (AGND), U3.2 (GND), U3.3 (NC), U3.4 (NC), U4.PAD (VSS)
- net BOOT0: no longer AP1.1, R20.1
- net PGND: now also NT3.1, NT7.1; no longer C1.2, C2.2, C3.2, C4.2
- net PH1: now also C6.2, R41.1
- net PWM1: now also U4.29 (PC6), U4.30 (PA8), C7.1, R37.1
- net PWM1N: now also U4.39 (PC10), C26.1
- net PWM2: now also U4.31 (PA9)
- net PWM3: now also U4.32 (PA10)
- net VM: now also R36.2
- net +VSENS1: now reaches U4.18 (PB1)
- net +VSENS1: now also C28.1, R39.1
- net VBAT: now reaches U4.38 (PA15)
- net VBAT: now also R36.1
- net at J2.2 (Pin_2): no longer U4.9 (PA1)
- net HO1 renamed HO
- net HO: no longer C6.2
- net HSE_IN: no longer names the net of U4.5 (PF0-OSC_IN)
- net HSE_OUT: no longer names the net of U4.6 (PF1-OSC_OUT)
- net ISENSE1 renamed +ISENS1
- net +ISENS1: now also U4.9 (PA1), TH1.1
- net LO1 renamed LO
- new net: NT2.3, U4.PAD (VSS)
- new net: R38.2, R39.2, R41.2
- new net: R29.2, R40.1, TH1.2
- new net: NT4.1, NT7.2
- new net: D1.1 (K), F1.1, J3.A4 (VBUS), J3.B4 (VBUS)
- new net: NT1.3, NT4.2
- new net: AP1.1, R20.1
- new net: NT2.1, NT5.2
- new net: NT1.1, NT2.2
- new net: NT6.1, NT8.1
- new net: J3.B5 (CC2), R35.1
- new net: NT5.3, NT6.2
- new net: NT3.2, R15.2
- new net: J3.A5 (CC1), R34.1
- new net: D7.2 (A), R33.2
- new net -ISENS1: NT1.2, NT3.3
- new net -ISENS2: NT4.3
- new net -ISENS3: NT7.3
- new net -VSENS1: NT5.1, R38.1
- new net -VSENS2: NT6.3
- new net -VSENS3: NT8.3
- new net GND: C1.2, C10.2, C11.2, C12.2, C15.2, C16.2, C17.2, C18.2, C2.2, C21.2, C22.2, C23.2, C24.2, C25.2, C26.2, C27.2, C28.2, C3.2, C4.2, C43.2, C44.2, C5.2, C7.2, C9.2, D1.2 (A), D4.1 (K), D6.1 (K), D7.1 (K), J1.5 (GND), J3.A1 (GND), J3.B1 (GND), J3.SH1 (SHIELD), J3.SH2 (SHIELD), J3.SH3 (SHIELD), J3.SH4 (SHIELD), NT8.2, R12.2, R13.2, R14.2, R20.2, R23.2, R25.2, R26.2, R32.2, R34.2, R35.2, R37.2, U1.7 (VSS), U1.PAD (VSS), U2.1 (AGND), U2.2 (PGND), U2.PAD (AGND), U3.2 (GND), U3.3 (NC), U3.4 (NC), U8.3 (GND)
- new net TSENS1: C27.1, R29.1
- new net USB_D+: J3.A6 (D1+), J3.B6 (D2+), U8.1 (D+)
- new net USB_D-: J3.A7 (D1-), J3.B7 (D2-), U8.2 (D-)
- new net USB_VBUS_SENSE: R31.2, R32.1
- new net VBUS: C43.1, C44.1, F1.2, R31.1, R33.1, TP4.1
- no-connect marks 1 -> 3
Other:
- note added: "CC1 and CC2 pulled down with 5.1k resistors => advertise USB devide mode --------- SBU1/2 for alternate DisplayPort mode --------- VBUS Sensing disabled"
- note added: "USB-C"
- note removed: "VOLTAGE SENSING A/B/C"
- moved on the sheet: AP1, C10, C11, C12, C2, C20, C22, C23, C24, C3, C4, C5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

Commit message: V1 schematic
Parts:
- removed C22, C23, C24, C26, C28, C7: 100p, Capacitor_SMD:C_0603_1608Metric, symbol ESC-SchemSymLib:CL10C101JB8NNNC
- removed C27: 100n, Capacitor_SMD:C_0402_1005Metric, symbol ESC-SchemSymLib:CL05B104KO5NNNC
- removed C5: 1u, Capacitor_SMD:C_0603_1608Metric, symbol ESC-SchemSymLib:CL10A105KB8NNNC
- removed C6: 220n, Capacitor_SMD:C_0402_1005Metric, symbol ESC-SchemSymLib:CL05B224KO5NNNC
- removed D2, D3, D5: RB161QS-40T18R, ESC-FootprintLib:Rohm_SMD1006, symbol ESC-SchemSymLib:RB161QS-40T18R
- removed J3: USB4105-GF-A, ESC-FootprintLib:GCT_USB4105-GF-A, symbol FC-SchemSymbolLib:USB4105-GF-A
- removed NT1, NT3, NT4, NT5, NT6, NT7, NT8: NetTie_3_Tee, symbol Device:NetTie_3_Tee
- removed NT2: NetTie_4_Cross, symbol Device:NetTie_4_Cross
- removed PH1: ~, TestPoint:TestPoint_Pad_4.0x4.0mm, symbol ESC-SchemSymLib:PhaseConnector
- removed Q1, Q2: CSD18540Q5B, ESC-FootprintLib:TRANS_CSD18540Q5B, symbol ESC-SchemSymLib:CSD18540Q5B
- removed R1, R3, R8: 3.3, Resistor_SMD:R_0402_1005Metric, symbol ESC-SchemSymLib:0402WGJ033JTCE
- removed R11, R2: 10, Resistor_SMD:R_0402_1005Metric, symbol ESC-SchemSymLib:0402WGF100JTCE
- removed R13, R16, R17, R30, R4, R40, R41: 10k, Resistor_SMD:R_0402_1005Metric, symbol ESC-SchemSymLib:0402WGF1002TCE
- removed R15: 0.5m, ESC-FootprintLib:Kelvin Shunt 1216 (3038), symbol ESC-SchemSymLib:HoBB1216-5W-0.5mR-1%
- removed R20, R37: 200k, Resistor_SMD:R_0402_1005Metric, symbol ESC-SchemSymLib:0402WGF2003TCE
- removed R21, R22, R24, R29, R39: 33, Resistor_SMD:R_0402_1005Metric, symbol ESC-SchemSymLib:0402WGF330JTCE
- removed R23, R25, R26, R38: 1k, Resistor_SMD:R_0402_1005Metric, symbol ESC-SchemSymLib:0402WGF1001TCE
- removed R31: 5.1k, Resistor_SMD:R_0402_1005Metric, symbol FC-SchemSymbolLib:0402WGF5101TCE
- removed R32: 10k, Resistor_SMD:R_0402_1005Metric, symbol FC-SchemSymbolLib:0402WGF1002TCE
- removed TH1: Thermistor_NTC, Resistor_SMD:R_0402_1005Metric, symbol ESC-SchemSymLib:NTCG103JF103FT1
- removed TP4: TestPoint, TestPoint:TestPoint_Pad_D1.0mm, symbol Connector:TestPoint
- removed U1: 2EDL8024, ESC-FootprintLib:2EDL8x2x_PG-VDSON-8-4, symbol ESC-SchemSymLib:2EDL8024
- added C29, C32, C33: 100p, Capacitor_SMD:C_0603_1608Metric, symbol ESC-SchemSymLib:CL10C101JB8NNNC
- added C30: 220n, Capacitor_SMD:C_0402_1005Metric, symbol ESC-SchemSymLib:CL05B224KO5NNNC
- added C31: 1u, Capacitor_SMD:C_0603_1608Metric, symbol ESC-SchemSymLib:CL10A105KB8NNNC
- added C34: 100n, Capacitor_SMD:C_0402_1005Metric, symbol ESC-SchemSymLib:CL05B104KO5NNNC
- added C41, C42: 10p, Capacitor_SMD:C_0402_1005Metric, symbol FC-SchemSymbolLib:CL05C100JB5NNNC
- added D10, D11, D12, D8, D9: RB161QS-40T18R, ESC-FootprintLib:Rohm_SMD1006, symbol ESC-SchemSymLib:RB161QS-40T18R
- added J3: USB4105-GF-A, ESC-FootprintLib:GCT_USB4105-GF-A, symbol ESC-SchemSymLib:USB4105-GF-A
- added NT1, NT10, NT11, NT12, NT13, NT14, NT2, NT3, NT4, NT5, NT6, NT7, NT8, NT9: NetTie_2, symbol ESC-SchemSymLib:NetTie_2
- added PH2: ~, TestPoint:TestPoint_Pad_4.0x4.0mm, symbol ESC-SchemSymLib:PhaseConnector
- added Q3, Q4: CSD18540Q5B, ESC-FootprintLib:TRANS_CSD18540Q5B, symbol ESC-SchemSymLib:CSD18540Q5B
- added R20, R44, R45, R50, R53: 10k, Resistor_SMD:R_0402_1005Metric, symbol ESC-SchemSymLib:0402WGF1002TCE
- added R31, R42, R47: 3.3, Resistor_SMD:R_0402_1005Metric, symbol ESC-SchemSymLib:0402WGJ033JTCE
- added R32, R48: 10, Resistor_SMD:R_0402_1005Metric, symbol ESC-SchemSymLib:0402WGF100JTCE
- added R43, R52: 33, Resistor_SMD:R_0402_1005Metric, symbol ESC-SchemSymLib:0402WGF330JTCE
- added R46: 1k, Resistor_SMD:R_0402_1005Metric, symbol ESC-SchemSymLib:0402WGF1001TCE
- added R49: 200k, Resistor_SMD:R_0402_1005Metric, symbol ESC-SchemSymLib:0402WGF2003TCE
- added R51: 0.5m, ESC-FootprintLib:Kelvin Shunt 1216 (3038), symbol ESC-SchemSymLib:HoBB1216-5W-0.5mR-1%
- added R68: 0R, Resistor_SMD:R_0402_1005Metric, symbol FC-SchemSymbolLib:0402WGF0000TCE
- added TH2: Thermistor_NTC, Resistor_SMD:R_0402_1005Metric, symbol ESC-SchemSymLib:NTCG103JF103FT1
- added U5: 2EDL8024, ESC-FootprintLib:2EDL8x2x_PG-VDSON-8-4, symbol ESC-SchemSymLib:2EDL8024
- added X2: 16MHz, Crystal:Crystal_SMD_2520-4Pin_2.5x2.0mm, symbol FC-SchemSymbolLib:X322516MLB4SI
Connections:
- net +3.3V is gone; now on net +3V3: C21.1, J1.1 (VCC), LED1.2, LED1.4, LED1.6
- net +3V3A is gone; now on net +3V3: C13.1, C14.1, U4.21 (VDDA)
- net +3V3REF is gone; now on net +3V3: C19.1, C20.1, U4.20 (VREF+)
- net AGND is gone; now on net GND: C13.2, C14.2, C19.2, C20.2
- net BOOT0 is gone; now on net PWM2: U4.46 (PB8-BOOT0)
- net MCU is gone; now on net GND: J2.3 (Pin_3)
- net VM is gone; now on net VBAT: C1.1, C2.1, C3.1, C4.1, R36.2, R5.1, R6.1, U2.3 (VIN)
- net +3V3: now also NT10.1, NT2.1, NT3.1, NT4.1, NT5.1, NT7.1, NT8.1, R53.2
- net +ISENS1: now also Q4.3 (S), R51.1, TH2.1
- net +VSENS1: now also C29.1, R43.1
- net -ISENS1: now also NT1.2, NT9.2, R51.2
- net GND: now also U4.PAD (VSS), C29.2, C31.2, C32.2, C33.2, C34.2, C41.2, C42.2, J3.A1 (GND), J3.B1 (GND), J3.SH1 (SHIELD), J3.SH2 (SHIELD), J3.SH3 (SHIELD), J3.SH4 (SHIELD), NT1.1, NT11.1, NT12.1, NT13.1, NT14.1, NT6.2, R20.1, R46.1, R49.2, R50.2, U5.7 (VSS), U5.PAD (VSS), X2.2, X2.4
- net HB1: now also C30.1, D10.1 (K), U5.2 (HB)
- net HO: now also D11.1 (K), R42.1, U5.3 (HO)
- net LO: now also D12.1 (K), R47.1, U5.8 (LO)
- net PGND: now also NT6.1, NT9.1
- net PH1: now also C30.2, PH2.1 (Pin_1), Q3.3 (S), Q4.1 (D), R44.2, R45.1, U5.4 (HS)
- net PWM1: now also C33.1, R49.1, U5.5 (HI); no longer U4.30 (PA8)
- net PWM1N: now also C32.1, U5.6 (LI)
- net PWM2: now also AP1.1, NT14.2; no longer U4.31 (PA9)
- net PWM3: now also U4.47 (PB9), NT12.2; no longer U4.32 (PA10)
- net RGB_LED_B: now also U4.2 (PC13)
- net RGB_LED_G: now also U4.3 (PC14-OSC32_IN)
- net RGB_LED_R: now also U4.4 (PC15-OSC32_OUT)
- net TSENS1: now also C34.1, R52.1
- net USB_D+: now also U4.34 (PA12), J3.A6 (D1+), J3.B6 (D2+)
- net USB_D-: now also U4.33 (PA11), J3.A7 (D1-), J3.B7 (D2-)
- net VBAT: now also Q3.1 (D); no longer R36.1, U4.38 (PA15)
- net +ISENS2: now reaches U4.15 (PA7)
- net +ISENS2: now also NT8.2
- net PWM2N: now reaches U4.22 (PB10)
- net PWM2N: now also NT13.2
- net +VSENS2: now reaches U4.25 (PB12)
- net +VSENS2: now also NT2.2
- net +TSENS2: now reaches U4.26 (PB13)
- net +TSENS2: now also NT3.2
- net +ISENS3: now reaches U4.27 (PB14)
- net +ISENS3: now also NT4.2
- net +TSENS3: now reaches U4.28 (PB15)
- net +TSENS3: now also NT5.2
- net PWM3N: now reaches U4.43 (PB5)
- net PWM3N: now also NT11.2
- net at U4.5 (PF0-OSC_IN): now also R68.1
- net at U4.6 (PF1-OSC_OUT): now also C41.1, X2.1
- net +TSENS1: now reaches U4.8 (PA0)
- net +TSENS1: now also NT10.2
- net at D1.1 (K), F1.1: now also J3.A4 (VBUS), J3.B4 (VBUS)
- net PWM/DSHOOT: now reaches J2.2 (Pin_2)
- net PWM/DSHOOT: now also U4.32 (PA10)
- net at R35.1: now also J3.B5 (CC2)
- net at R34.1: now also J3.A5 (CC1)
- net +10.5V renamed VBUCK
- net VBUCK: now also C31.1, D9.2 (A), R31.1, U5.1 (VDD); no longer C9.1, U3.1 (VIN)
- net +10.5VNoise: no longer names the net of C8.1, L1.1, U2.11 (SW), U2.12 (SW)
- net VBUS renamed +5V
- net +5V: now also D8.2 (A)
- new net: C42.1, R68.2, X2.3
- new net: D10.2 (A), R31.2
- new net: C9.1, D8.1 (K), D9.1 (K), U3.1 (VIN)
- new net: R43.2, R45.2, R46.2
- new net: R52.2, R53.1, TH2.2
- new net: Q4.2 (G), R47.2, R48.2, R50.1
- new net: Q3.2 (G), R32.2, R42.2, R44.1
- new net: D11.2 (A), R32.1
- new net: D12.2 (A), R48.1
- new net +VSENS3: NT7.2, U4.30 (PA8)
- new net VSENSBAT: R20.2, R36.1, U4.38 (PA15)
- no-connect marks 3 -> 17
Other:
- note added: "3V3 LDO"
- note added: "MCU"
- note added: "SPEED CONTROL"
- note removed: "10V to 3V3 LDO"
- note removed: "CC1 and CC2 pulled down with 5.1k resistors => advertise USB devide mode --------- SBU1/2 for alternate DisplayPort mode --------- VBUS Sensing disabled"
- note removed: "Must be placed near MCU ADC pins."
- moved on the sheet: AP1, C1, C10, C11, C12, C13, C14, C15, C16, C17, C18, C19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

Commit message: First PCB
Parts:
- removed C11, C12: 1u, Capacitor_SMD:C_0603_1608Metric, symbol ESC-SchemSymLib:CL10A105KB8NNNC
- removed D7: LED, LED_SMD:LED_0603_1608Metric, symbol Device:LED
- removed J2: Conn_01x03_Socket, symbol Connector:Conn_01x03_Socket
- removed R33: 220, Resistor_SMD:R_0402_1005Metric, symbol FC-SchemSymbolLib:0402WGF2200TCE
- added C11, C5, C6, C7: 1u, Capacitor_SMD:C_0402_1005Metric, symbol FC-SchemSymbolLib:CL05A105KA5NQNC
- added D2: KT-0603W, LED_SMD:LED_0603_1608Metric, symbol ESC-SchemSymLib:KT-0603W
- added IN1, IN2: ~, TestPoint:TestPoint_Pad_2.0x2.0mm, symbol ESC-SchemSymLib:InputConnector
- added NT15: NetTie_2, NetTie:NetTie-2_SMD_Pad0.5mm, symbol ESC-SchemSymLib:NetTie_2
- added PH4: ~, TestPoint:TestPoint_Pad_4.0x4.0mm, symbol ESC-SchemSymLib:PhaseConnector
- added R1: 1k, Resistor_SMD:R_0402_1005Metric, symbol ESC-SchemSymLib:0402WGF1001TCE
- NT1, NT10, NT11, NT12, NT13, NT14, NT2, NT3, NT4, NT5, NT6, NT7, NT8, NT9: footprint (none) -> NetTie:NetTie-2_SMD_Pad0.5mm
- U2: footprint Package_SON:WSON-12-1EP_4x4mm_P0.5mm_EP2.6x3mm -> ESC-FootprintLib:WSON-12-1EP_4x4mm_P0.5mm_EP2.6x3mm
- U4: footprint Package_DFN_QFN:QFN-48-1EP_7x7mm_P0.5mm_EP5.6x5.6mm_ThermalVias -> ESC-FootprintLib:QFN-48-1EP_7x7mm_P0.5mm_EP5.6x5.6mm
Connections:
- net +5V: now also R1.1
- net GND: now also C11.2, C5.2, C6.2, C7.2, D2.1 (K), NT15.2
- net PGND: now also PH2.1 (Pin_1)
- net PH1: no longer PH2.1 (Pin_1)
- net PWM/DSHOOT: now also IN1.1 (Pin_1)
- net VBAT: now also C5.1, C7.1, PH4.1 (Pin_1)
- net VIN: now reaches C9.1, D8.1 (K), D9.1 (K), U3.1 (VIN)
- net SW: now reaches C8.1, L1.1, U2.11 (SW), U2.12 (SW)
- net at U2.6 (SS): now also C11.1
- net at U2.7 (FPWM): no longer U2.9 (VCC)
- net VBUS: now reaches D1.1 (K), F1.1, J3.A4 (VBUS), J3.B4 (VBUS)
- new net: D2.2 (A), R1.2
- new net: C6.1, U2.9 (VCC)
- new net GND_FC: IN2.1 (Pin_1), NT15.1
Other:
- note added: "BATTERY INPUT"
- note added: "SPEED INPUT"
- note removed: "SPEED CONTROL"
- moved on the sheet: C1, C2, C3, C4, C9, D9, R20, R36, R5
