File: hardware/KiCad/ESC_v1.0/ESC_v1.0.kicad_sch (KiCad schematic)
At the start: 105 parts, among them J1 Conn_ARM_SWD_TagConnect_TC203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, J3 USB4105-GF-A, Q3 CSD18540Q5B, Q4 CSD18540Q5B, U2 LM5160A, U3 TPS7B92033, U4 STM32G484CEU6, U5 2EDL8024, U8 TPD2EUSB30A, X2 16MHz

Commit message: PCB
Connections:
- net GND: no longer C1.2, C2.2, C3.2, C4.2
- net PGND: now also C1.2, C2.2, C3.2, C4.2
- net GL1: now reaches Q4.2 (G), R47.2, R48.2, R50.1
- net GH1: now reaches Q3.2 (G), R32.2, R42.2, R44.1
- net HO renamed HO1
- net LO renamed LO1
Changed lines of the file:
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@@
 	)
 	(junction
-		(at 328.93 124.46)
-		(diameter 0)
-		(color 0 0 0 0)
-	)
-	(junction
 		(at 104.14 168.91)
 		(diameter 0)
@@
 	)
 	(junction
-		(at 190.5 34.29)
-		(diameter 0)
-		(color 0 0 0 0)
-	)
-	(junction
 		(at 146.05 80.01)
 		(diameter 0)
@@
 	)
 	(junction
+		(at 190.5 34.29)
+		(diameter 0)
+		(color 0 0 0 0)
+	)
+	(junction
 		(at 344.17 124.46)
 		(diameter 0)
@@
 	)
 	(junction
+		(at 328.93 124.46)
+		(diameter 0)
+		(color 0 0 0 0)
+	)
+	(junction
 		(at 203.2 26.67)
 		(diameter 0)
@@
 	(wire
 		(pts
-			(xy 339.09 124.46) (xy 328.93 124.46)
-		)
-		(stroke
-			(width 0)
-			(type default)
-		)
-	)
-	(wire
-		(pts
 			(xy 86.36 262.89) (xy 88.9 262.89)
 		)
@@
 	(wire
 		(pts
+			(xy 328.93 116.84) (xy 331.47 116.84)
+		)
+		(stroke
+			(width 0)
+			(type default)
+		)
+	)
+	(wire
+		(pts
 			(xy 339.09 153.67) (xy 339.09 152.4)
 		)
@@
 	(wire
 		(pts
+			(xy 328.93 124.46) (xy 339.09 124.46)
+		)
+		(stroke
+			(width 0)
+			(type default)
+		)
+	)
+	(wire
+		(pts
 			(xy 41.91 229.87) (xy 44.45 229.87)
 		)
@@
 	(wire
 		(pts
-			(xy 328.93 116.84) (xy 331.47 116.84)
-		)
-		(stroke
-			(width 0)
-			(type default)
-		)
-	)
-	(wire
-		(pts
 			(xy 82.55 262.89) (xy 83.82 262.89)
 		)
@@
 		)
 	)
-	(label "HO"
+	(label "HO1"
 		(at 297.18 121.92 0)
 		(effects
@@
 		)
 	)
-	(label "LO"
+	(label "LO1"
 		(at 297.18 127 0)
 		(effects
@@
 		)
 	)
+	(label "GL1"
+		(at 328.93 132.08 180)
+		(effects
+			(font
+				(size 1 1)
+			)
+			(justify right bottom)
+		)
+	)
 	(label "+ISENS3"
 		(at 125.73 261.62 180)
@@
 		)
 	)
+	(label "GH1"
+		(at 328.93 116.84 180)
+		(effects
+			(font
+				(size 1 1)
+			)
+			(justify right bottom)
+		)
+	)
 	(label "VIN"
 		(at 124.46 124.46 0)
@@
 	)
 	(symbol
+		(lib_id "power:GND")
+		(at 190.5 34.29 0)
+		(mirror y)
+		(unit 1)
+		(exclude_from_sim no)
+		(in_bom yes)
+		(on_board yes)
+		(dnp no)
+		(property "Reference" "#PWR018"
+			(at 190.5 40.64 0)
+			(effects
+				(font
+					(size 1.27 1.27)
+				)
+				(hide yes)
+			)
+		)
+		(property "Value" "PGND"
+			(at 190.5 38.608 0)
+			(effects
+				(font
+					(size 1.27 1.27)
+				)
+			)
+		)
+		(property "Footprint" ""
+			(at 190.5 34.29 0)
+			(effects
+				(font
+					(size 1.27 1.27)
+				)
+				(hide yes)
+			)
+		)
+		(property "Datasheet" ""
+			(at 190.5 34.29 0)
+			(effects
+				(font
+					(size 1.27 1.27)
+				)
+				(hide yes)
+			)
+		)
+		(property "Description" "Power symbol creates a global label with name \"GND\" , ground"
+			(at 190.5 34.29 0)
+			(effects
+				(font
+					(size 1.27 1.27)
+				)
+				(hide yes)
+			)
+		)
+		(pin "1"
+		)
+		(instances
+			(project "ESC_v1.0"
+				(path "/30189dae-47a7-45f4-9b84-2dfd500c2612"
+					(reference "#PWR018")
+					(unit 1)
+				)
+			)
+		)
+	)
+	(symbol
 		(lib_id "FC-SchemSymbolLib:X322516MLB4SI")
 		(at 134.62 227.33 0)
@@
 	)
 	(symbol
-		(lib_id "power:GND")
-		(at 181.61 41.91 0)
-		(mirror y)
-		(unit 1)
-		(exclude_from_sim no)
-		(in_bom yes)
-		(on_board yes)
-		(dnp no)
-		(fields_autoplaced yes)
-		(property "Reference" "#PWR35"
-			(at 181.61 48.26 0)
-			(effects
-				(font
-					(size 1.27 1.27)
-				)
-				(hide yes)
-			)
-		)
-		(property "Value" "GND"
-			(at 181.61 46.99 0)
-			(effects
-				(font
-					(size 1.27 1.27)
-				)
-				(hide yes)
-			)
-		)
-		(property "Footprint" ""
-			(at 181.61 41.91 0)
-			(effects
-				(font
-					(size 1.27 1.27)
-				)
-				(hide yes)
-			)
-		)
-		(property "Datasheet" ""
-			(at 181.61 41.91 0)
-			(effects
-				(font
-					(size 1.27 1.27)
-				)
-				(hide yes)
-			)
-		)
-		(property "Description" "Power symbol creates a global label with name \"GND\" , ground"
-			(at 181.61 41.91 0)
-			(effects
-				(font
-					(size 1.27 1.27)
-				)
-				(hide yes)
-			)
-		)
-		(pin "1"
-		)
-		(instances
-			(project "ESC_v1.0"
-				(path "/30189dae-47a7-45f4-9b84-2dfd500c2612"
-					(reference "#PWR35")
-					(unit 1)
-				)
-			)
-		)
-	)
-	(symbol
 		(lib_id "power:+3V3")
 		(at 368.3 152.4 90)
@@
 	(symbol
 		(lib_id "power:GND")
-		(at 190.5 34.29 0)
+		(at 181.61 41.91 0)
 		(mirror y)
 		(unit 1)
@@
 		(fields_autoplaced yes)
 		(property "Reference" "#PWR43"
-			(at 190.5 40.64 0)
+			(at 181.61 48.26 0)
 			(effects
 				(font
@@
 		)
 		(property "Value" "GND"
-			(at 190.5 39.37 0)
+			(at 181.61 46.99 0)
 			(effects
 				(font
@@
 		)
 		(property "Footprint" ""
-			(at 190.5 34.29 0)
+			(at 181.61 41.91 0)
 			(effects
 				(font
@@
 		)
 		(property "Datasheet" ""
-			(at 190.5 34.29 0)
+			(at 181.61 41.91 0)
 			(effects
 				(font
@@
 		)
 		(property "Description" "Power symbol creates a global label with name \"GND\" , ground"
-			(at 190.5 34.29 0)
+			(at 181.61 41.91 0)
 			(effects
 				(font

Commit message: Major board update
Parts:
- removed AP1: ActionPad, TestPoint:TestPoint_Pad_1.5x1.5mm, symbol ESC-SchemSymLib:ActionPad
- removed C10, C15: 4.7u, Capacitor_SMD:C_0805_2012Metric, symbol ESC-SchemSymLib:CL21A475KAQNNNE
- removed C16, C18, C19, C25, C34: 100n, Capacitor_SMD:C_0402_1005Metric, symbol ESC-SchemSymLib:CL05B104KO5NNNC
- removed C20, C31, C9: 1u, Capacitor_SMD:C_0603_1608Metric, symbol ESC-SchemSymLib:CL10A105KB8NNNC
- removed C29, C32, C33: 100p, Capacitor_SMD:C_0603_1608Metric, symbol ESC-SchemSymLib:CL10C101JB8NNNC
- removed C30: 220n, Capacitor_SMD:C_0402_1005Metric, symbol ESC-SchemSymLib:CL05B224KO5NNNC
- removed C43: 1u, Capacitor_SMD:C_0402_1005Metric, symbol FC-SchemSymbolLib:CL05A105KA5NQNC
- removed C44: 100n, Capacitor_SMD:C_0402_1005Metric, symbol FC-SchemSymbolLib:CL05B104KO5NNNC
- removed D1: ESD5Zxx, Diode_SMD:D_SOD-523, symbol Diode:ESD5Zxx
- removed D10, D11, D12, D8, D9: RB161QS-40T18R, ESC-FootprintLib:Rohm_SMD1006, symbol ESC-SchemSymLib:RB161QS-40T18R
- removed D2: KT-0603W, LED_SMD:LED_0603_1608Metric, symbol ESC-SchemSymLib:KT-0603W
- removed F1: Polyfuse, Resistor_SMD:R_1812_4532Metric, symbol Device:Polyfuse
- removed IN1, IN2: ~, TestPoint:TestPoint_Pad_2.0x2.0mm, symbol ESC-SchemSymLib:InputConnector
- removed J1: Conn_ARM_SWD_TagConnect_TC2030-NL, Connector:Tag-Connect_TC2030-IDC-NL_2x03_P1.27mm_Vertical, symbol Connector:Conn_ARM_SWD_TagConnect_TC2030-NL
- removed J3: USB4105-GF-A, ESC-FootprintLib:GCT_USB4105-GF-A, symbol ESC-SchemSymLib:USB4105-GF-A
- removed NT1, NT10, NT11, NT12, NT13, NT14, NT15, NT2, NT3, NT4, NT5, NT6, NT7, NT8, NT9: NetTie_2, NetTie:NetTie-2_SMD_Pad0.5mm, symbol ESC-SchemSymLib:NetTie_2
- removed PH2, PH4: ~, TestPoint:TestPoint_Pad_4.0x4.0mm, symbol ESC-SchemSymLib:PhaseConnector
- removed Q3, Q4: CSD18540Q5B, ESC-FootprintLib:TRANS_CSD18540Q5B, symbol ESC-SchemSymLib:CSD18540Q5B
- removed R1, R46: 1k, Resistor_SMD:R_0402_1005Metric, symbol ESC-SchemSymLib:0402WGF1001TCE
- removed R31, R42, R47: 3.3, Resistor_SMD:R_0402_1005Metric, symbol ESC-SchemSymLib:0402WGJ033JTCE
- removed R32, R48: 10, Resistor_SMD:R_0402_1005Metric, symbol ESC-SchemSymLib:0402WGF100JTCE
- removed R34, R35: 5.1k, Resistor_SMD:R_0402_1005Metric, symbol FC-SchemSymbolLib:0402WGF5101TCE
- removed R43, R52: 33, Resistor_SMD:R_0402_1005Metric, symbol ESC-SchemSymLib:0402WGF330JTCE
- removed R44, R45, R50, R53: 10k, Resistor_SMD:R_0402_1005Metric, symbol ESC-SchemSymLib:0402WGF1002TCE
- removed R49: 200k, Resistor_SMD:R_0402_1005Metric, symbol ESC-SchemSymLib:0402WGF2003TCE
- removed R51: 0.5m, ESC-FootprintLib:Kelvin Shunt 1216 (3038), symbol ESC-SchemSymLib:HoBB1216-5W-0.5mR-1%
- removed R68: 0R, Resistor_SMD:R_0402_1005Metric, symbol FC-SchemSymbolLib:0402WGF0000TCE
- removed U4: STM32G484CEU6, ESC-FootprintLib:QFN-48-1EP_7x7mm_P0.5mm_EP5.6x5.6mm, symbol ESC-SchemSymLib:STM32G484CEU6
- removed U5: 2EDL8024, ESC-FootprintLib:2EDL8x2x_PG-VDSON-8-4, symbol ESC-SchemSymLib:2EDL8024
- removed U8: TPD2EUSB30A, Package_TO_SOT_SMD:Texas_DRT-3, symbol Power_Protection:TPD2EUSB30A
- added C1, C23, C7: 1u, Capacitor_SMD:C_0402_1005Metric, symbol ESC-SchemSymLib:CL05A105KA5NQNC
- added C15, C2, C24, C37: 100n, Capacitor_SMD:C_0402_1005Metric, symbol ESC-SchemSymLib:CL05B104KO5NNNC
- added C8: 2.2u, Capacitor_SMD:C_1206_3216Metric, symbol ESC-SchemSymLib:CL31B225KBHNNNE
- added D14, D2: RB161QS-40T18R, ESC-FootprintLib:Rohm_SMD1006, symbol ESC-SchemSymLib:RB161QS-40T18R
- added J1, J2: Conn_01x01, ESC-FootprintLib:Phase4x4, symbol Connector_Generic:Conn_01x01
- added J10, J3, J4, J5, J6: Conn_01x01, TestPoint:TestPoint_Pad_2.0x2.0mm, symbol Connector_Generic:Conn_01x01
- added J11: JTAG_TC2030, Connector:Tag-Connect_TC2030-IDC-NL_2x03_P1.27mm_Vertical, symbol ESC-SchemSymLib:Conn_ARM_SWD_TagConnect_TC2030-NL
- added R12: 10k, Resistor_SMD:R_0402_1005Metric, symbol ESC-SchemSymLib:0402WGF1002TCE
- added R13: 33, Resistor_SMD:R_0402_1005Metric, symbol ESC-SchemSymLib:0402WGF330JTCE
- added TP1, TP10, TP11, TP12, TP13, TP14, TP15, TP2, TP4, TP5, TP6, TP7, TP8, TP9: TestPoint, TestPoint:TestPoint_Pad_D1.0mm, symbol Connector:TestPoint
- added U1: STM32G484CEU6, ESC-FootprintLib:QFN-48-1EP_7x7mm_P0.5mm_EP5.6x5.6mm, symbol ESC-SchemSymLib:STM32G484CEU6
- C12: renamed from C7; symbol FC-SchemSymbolLib:CL05A105KA5NQNC -> ESC-SchemSymLib:CL05A105KA5NQNC
- C13: renamed from C5; symbol FC-SchemSymbolLib:CL05A105KA5NQNC -> ESC-SchemSymLib:CL05A105KA5NQNC
- C16: renamed from C6; symbol FC-SchemSymbolLib:CL05A105KA5NQNC -> ESC-SchemSymLib:CL05A105KA5NQNC
- C17: renamed from C11; symbol FC-SchemSymbolLib:CL05A105KA5NQNC -> ESC-SchemSymLib:CL05A105KA5NQNC
- C20: renamed from C42; symbol FC-SchemSymbolLib:CL05C100JB5NNNC -> ESC-SchemSymLib:CL05C100JB5NNNC; Distributor Link 1 (none) -> https://au.mouser.com/ProductDetail/Samsung-Electro-Mechani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; Distributor Link 2 (none) -> https://www.digikey.com/en/products/detail/samsung-electro-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
- C21: renamed from C41; symbol FC-SchemSymbolLib:CL05C100JB5NNNC -> ESC-SchemSymLib:CL05C100JB5NNNC; Distributor Link 1 (none) -> https://au.mouser.com/ProductDetail/Samsung-Electro-Mechani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; Distributor Link 2 (none) -> https://www.digikey.com/en/products/detail/samsung-electro-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
- X1: renamed from X2; symbol FC-SchemSymbolLib:X322516MLB4SI -> ESC-SchemSymLib:X322516MLB4SI; Distributor Link 1 (none) -> https://www.lcsc.com/product-detail/C13738.html; Distributor Link 2 (none) -> https://www.pcbx.com/component-detail/X322516MLB4SI-Yangxin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
- renumbered C17 to C11, C8 to C14, C13 to C18, C14 to C19, C21 to C25, C1 to C3, C2 to C4, C3 to C5, C4 to C6, D6 to D1, R36 to R1, R7 to R11, R28 to R14, R27 to R15, R18 to R16, R19 to R17, R20 to R2, R5 to R3, R6 to R4, R10 to R5, R9 to R6, R12 to R7, R14 to R8, TH2 to TH1
Connections:
- net PGND is gone; now on net GND: C3.2, C4.2, C5.2, C6.2
- net VIN is gone; now on net VBUCK: U3.1 (VIN)
- net GND: now also TH1.2, C1.2, C15.2, C2.2, C23.2, C24.2, C37.2, C7.1, C8.2, J11.5 (GND), J2.1 (Pin_1), J6.1 (Pin_1), TP10.1, U1.PAD (VSS)
- net PWM1: now also U1.32 (PA10)
- net PWM1N: now also U1.47 (PB9)
- net PWM2: now also U1.31 (PA9)
- net PWM2N: now also U1.27 (PB14)
- net PWM3: now also TP8.1, U1.30 (PA8)
- net PWM3N: now also TP7.1, U1.2 (PC13)
- net VBAT: now also C8.1, J1.1 (Pin_1), TP9.1
- net VBUCK: now also C23.1, TP12.1
- net VSENSBAT: now also TP15.1, U1.28 (PB15)
- net HSE_OUT: now reaches C21.1, X1.1
- net HSE_OUT: now also U1.6 (PF1-OSC_OUT)
- net HSE_IN: now reaches C20.1, X1.3
- net HSE_IN: now also U1.5 (PF0-OSC_IN)
- net UVLO: now reaches R4.2, R7.1, U2.4 (EN/UVLO)
- net RON: now reaches R3.2, U2.5 (RON)
- net SS: now reaches C17.1, U2.6 (SS)
- net FB: now reaches R6.2, R8.1, U2.8 (FB)
- net VCC: now reaches C16.1, U2.9 (VCC)
- net +3V3 renamed 3V3
- net 3V3: now also C15.1, C2.1, C37.1, C7.2, D14.1 (K), D2.1 (K), J11.1 (VCC), R12.1, TP14.1, U1.1 (VBAT), U1.20 (VREF+), U1.21 (VDDA), U1.23 (VDD), U1.35 (VDD), U1.48 (VDD); no longer R11.1, U3.5 (OUT)
- net +ISENS1: no longer names the net of TH1.1
- net +ISENS1: now also R12.2, R13.2
- net LED_B_K: no longer names the net of LED1.5, R17.2
- net LED_G_K: no longer names the net of LED1.3, R16.2
- net LED_R_K: no longer names the net of LED1.1, R15.1
- net RGB_LED_B renamed RGB_B
- net RGB_B: now also U1.42 (PB4)
- net RGB_LED_G renamed RGB_G
- net RGB_G: now also U1.40 (PC11)
- net RGB_LED_R renamed RGB_R
- net RGB_R: now also U1.43 (PB5)
- new net 3V3_LDO: C1.1, D2.2 (A), R11.1, U3.5 (OUT)
- new net 3V3_UART: D14.2 (A), J10.1 (Pin_1)
- new net BOOT0: TP1.1, U1.46 (PB8-BOOT0)
- new net ISENS1+: U1.17 (PB0)
- new net ISENS1-: U1.19 (PB2)
- new net ISENS1_OPAMP_VOUT: TP2.1, U1.10 (PA2)
- new net ISENS2+: U1.15 (PA7)
- new net ISENS2-: U1.13 (PA5)
- new net ISENS3+: TP5.1, U1.9 (PA1)
- new net ISENS3-: TP6.1, U1.11 (PA3)
- new net JTAG_NRST: J11.3 (~{RESET}), U1.7 (PG10-NRST)
- new net PH3: TP11.1
- new net SWCLK: J11.4 (SWCLK), U1.37 (PA14)
- new net SWDIO: J11.2 (SWDIO), U1.36 (PA13)
- new net SWO: J11.6 (SWO), U1.41 (PB3)
- new net THROTTLE_CMD: J5.1 (Pin_1), TP13.1, U1.38 (PA15)
- new net TSENS: C24.1, R13.1, U1.8 (PA0)
- new net UART_RX: J3.1 (Pin_1), U1.45 (PB7)
- new net UART_TX: J4.1 (Pin_1), U1.44 (PB6)
- new net VSENS1: U1.26 (PB13)
- new net VSENS2: U1.25 (PB12)
- new net VSENS3: TP4.1, U1.18 (PB1)
- no-connect marks 17 -> 12
Other:
- added sheet PHASE 1 (phase.kicad_sch)
- added sheet PHASE 2 (phase.kicad_sch)
- added sheet PHASE 3 (phase.kicad_sch)
- note added: "${REVISION}"
- note added: "Crystal"
- note added: "ESC Dev Board -"
- note added: "JTAG"
- note added: "Kururugi"
- note added: "TEMP SENSING"
- note added: "THROTTLE"
- note added: "UART"
- note added: "VM to VBUCK"
- note removed: "DEBUG Tag Connect"
- note removed: "Internal NRESET Pullup resistor already included in the MCU"
- note removed: "MCU"
- note removed: "PHASE 1"
- note removed: "SPEED INPUT"
- note removed: "USB-C"
- note removed: "VBAT FILTERING"
- note removed: "VM to 10.5V BUCK"
- moved on the sheet: C11, C12, C13, C14, C16, C17, C18, C19, C20, C21, C25, C3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

Commit message: Major Kicad Update
Parts:
- removed TP13: TestPoint, TestPoint:TestPoint_Pad_D1.0mm, symbol Connector:TestPoint
- added TP13: TestPoint, ESC-FootprintLib:TestPoint_Pad_D1.0mm, symbol ESC-SchemSymLib:TestPoint
- J1, J2: symbol Connector_Generic:Conn_01x01 -> ESC-SchemSymLib:Conn_01x01_Phase; now in the parts list
- J10, J3, J4, J5, J6: footprint TestPoint:TestPoint_Pad_2.0x2.0mm -> ESC-FootprintLib:TestPoint_Pad_2.0x2.0mm; symbol Connector_Generic:Conn_01x01 -> ESC-SchemSymLib:Conn_01x01; now in the parts list
- J11: footprint Connector:Tag-Connect_TC2030-IDC-NL_2x03_P1.27mm_Vertical -> ESC-FootprintLib:Tag-Connect_TC2030-IDC-NL_2x03_P1.27mm_Vertical
- TP1, TP11, TP12, TP14, TP15, TP2, TP4, TP5, TP6, TP7, TP8, TP9: footprint TestPoint:TestPoint_Pad_D1.0mm -> ESC-FootprintLib:TestPoint_Pad_D1.0mm; symbol Connector:TestPoint -> ESC-SchemSymLib:TestPoint; now in the parts list
- TP10: footprint TestPoint:TestPoint_Pad_D1.0mm -> ESC-FootprintLib:TestPoint_Pad_D1.0mm; symbol Connector:TestPoint -> ESC-SchemSymLib:TestPoint
Connections:
- net GND: now also TP13.1
Other:
- moved on the sheet: TP11
