File: hardware/KiCad/ESC_v1.0/ESC_v1.0.kicad_sch (KiCad schematic)
At the start: 71 parts, among them J1 Conn_01x01, J10 Conn_01x01, J11 JTAG_TC2030, J2 Conn_01x01, J3 Conn_01x01, J4 Conn_01x01, J5 Conn_01x01, J6 Conn_01x01, U1 STM32G484CEU6, U2 LM5160A, U3 TPS7B92033, X1 16MHz

Commit message: Fix Kicad
Parts:
- renumbered C2 to C1, C13 to C10, C14 to C11, C15 to C12, C16 to C13, C17 to C14, C18 to C15, C19 to C16, C7 to C17, C20 to C18, C21 to C19, C37 to C2, C1 to C20, C23 to C21, C24 to C22, C25 to C23, C8 to C7, C11 to C8, C12 to C9, D14 to D2, D2 to D3, J10 to J5, J11 to J6, J5 to J7, J6 to J8, R12 to R10, R13 to R11, R14 to R12, R15 to R13, R16 to R14, R17 to R15, R11 to R9, TP6 to TP10, TP12 to TP11, TP4 to TP12, TP11 to TP13, TP9 to TP2, TP10 to TP3, TP13 to TP4, TP7 to TP5, TP8 to TP6, TP5 to TP7, TP15 to TP8, TP2 to TP9
Other:
- moved on the sheet: C10, C17, C3, C4, C5, C6, C7, C9, D1, J6, R1, R2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

Commit message: Update documentation
Parts:
- C1, C12, C2, C22, C23, C8: symbol ESC-SchemSymLib:CL05B104KO5NNNC -> KururugiESC-Symbols-Lib:CL05B104KO5NNNC
- C10, C13, C14, C17, C20, C21, C9: symbol ESC-SchemSymLib:CL05A105KA5NQNC -> KururugiESC-Symbols-Lib:CL05A105KA5NQNC
- C11, C15: symbol ESC-SchemSymLib:CL05B103KB5NNNC -> KururugiESC-Symbols-Lib:CL05B103KB5NNNC
- C16: symbol ESC-SchemSymLib:CL10A105KB8NNNC -> KururugiESC-Symbols-Lib:CL10A105KB8NNNC
- C18, C19: symbol ESC-SchemSymLib:CL05C100JB5NNNC -> KururugiESC-Symbols-Lib:CL05C100JB5NNNC
- C3, C4, C5, C6, C7: symbol ESC-SchemSymLib:CL31B225KBHNNNE -> KururugiESC-Symbols-Lib:CL31B225KBHNNNE
- D1, D4: symbol ESC-SchemSymLib:KT-0603W -> KururugiESC-Symbols-Lib:KT-0603W
- D2, D3: symbol ESC-SchemSymLib:RB161QS-40T18R -> KururugiESC-Symbols-Lib:RB161QS-40T18R
- J1: symbol ESC-SchemSymLib:Conn_01x01_Phase -> KururugiESC-Symbols-Lib:Conn_01x01_Phase_1
- J2: symbol ESC-SchemSymLib:Conn_01x01_Phase -> KururugiESC-Symbols-Lib:Conn_01x01_Phase
- J3: symbol ESC-SchemSymLib:Conn_01x01 -> KururugiESC-Symbols-Lib:Conn_01x01
- J4: symbol ESC-SchemSymLib:Conn_01x01 -> KururugiESC-Symbols-Lib:Conn_01x01_4
- J5: symbol ESC-SchemSymLib:Conn_01x01 -> KururugiESC-Symbols-Lib:Conn_01x01_3
- J6: symbol ESC-SchemSymLib:Conn_ARM_SWD_TagConnect_TC2030-NL -> KururugiESC-Symbols-Lib:Conn_ARM_SWD_TagConnect_TC2030-NL
- J7: symbol ESC-SchemSymLib:Conn_01x01 -> KururugiESC-Symbols-Lib:Conn_01x01_1
- J8: symbol ESC-SchemSymLib:Conn_01x01 -> KururugiESC-Symbols-Lib:Conn_01x01_2
- L1: symbol ESC-SchemSymLib:LVS404018-220M-N -> KururugiESC-Symbols-Lib:LVS404018-220M-N
- LED1: symbol ESC-SchemSymLib:LED_19-337C -> KururugiESC-Symbols-Lib:LED_19-337C
- R1, R10, R2: symbol ESC-SchemSymLib:0402WGF1002TCE -> KururugiESC-Symbols-Lib:0402WGF1002TCE
- R11: symbol ESC-SchemSymLib:0402WGF330JTCE -> KururugiESC-Symbols-Lib:0402WGF330JTCE
- R12, R13, R14, R15, R9: symbol ESC-SchemSymLib:0402WGF1000TCE -> KururugiESC-Symbols-Lib:0402WGF1000TCE
- R3: symbol ESC-SchemSymLib:0603WAF1203T5E -> KururugiESC-Symbols-Lib:0603WAF1203T5E
- R4: symbol ESC-SchemSymLib:0402WGF2003TCE -> KururugiESC-Symbols-Lib:0402WGF2003TCE
- R5: symbol ESC-SchemSymLib:0402WGF1001TCE -> KururugiESC-Symbols-Lib:0402WGF1001TCE
- R6: symbol ESC-SchemSymLib:0402WGF5102TCE -> KururugiESC-Symbols-Lib:0402WGF5102TCE
- R7: symbol ESC-SchemSymLib:0402WGF2202TCE -> KururugiESC-Symbols-Lib:0402WGF2202TCE
- R8: symbol ESC-SchemSymLib:0402WGF1202TCE -> KururugiESC-Symbols-Lib:0402WGF1202TCE
- TH1: symbol ESC-SchemSymLib:NTCG103JF103FT1 -> KururugiESC-Symbols-Lib:NTCG103JF103FT1
- TP1, TP10, TP11, TP12, TP13, TP14, TP2, TP3, TP4, TP5, TP6, TP7, TP8, TP9: symbol ESC-SchemSymLib:TestPoint -> KururugiESC-Symbols-Lib:TestPoint
- U1: symbol ESC-SchemSymLib:STM32G484CEU6 -> KururugiESC-Symbols-Lib:STM32G484CEU6
- U2: symbol ESC-SchemSymLib:LM5160ADNTR -> KururugiESC-Symbols-Lib:LM5160ADNTR
- U3: symbol ESC-SchemSymLib:TPS7B92033 -> KururugiESC-Symbols-Lib:TPS7B92033
- X1: symbol ESC-SchemSymLib:X322516MLB4SI -> KururugiESC-Symbols-Lib:X322516MLB4SI
Other:
- note added: "CRYSTAL"
- note added: "VGATE BUCK"
- note removed: "Crystal"
- note removed: "VM to VBUCK"
