File: hardware/KiCad/ESC_v1.0/phase.kicad_sch (KiCad schematic)
At the start: 21 parts, among them J7 Conn_01x01, Q1 CSD18540Q5B, Q2 CSD18540Q5B, U4 2EDL8024

Commit message: Major Kicad Update
Parts:
- J7: symbol Connector_Generic:Conn_01x01 -> ESC-SchemSymLib:Conn_01x01_Phase; now in the parts list
Changed lines of the file:
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@@
 	)
 	(symbol
-		(lib_name "HoBB1216-5W-0.5mR-1%_1")
 		(lib_id "ESC-SchemSymLib:HoBB1216-5W-0.5mR-1%")
 		(at 148.59 115.57 0)
@@
 	)
 	(symbol
-		(lib_name "Conn_01x01_7")
-		(lib_id "Connector_Generic:Conn_01x01")
+		(lib_id "ESC-SchemSymLib:Conn_01x01_Phase")
 		(at 217.17 69.85 0)
 		(mirror x)
 		(unit 1)
 		(exclude_from_sim no)
-		(in_bom no)
+		(in_bom yes)
 		(on_board yes)
 		(dnp no)
@@
 			)
 		)
-		(property "Description" "Connector for x1 motor phase wire."
+		(property "Description" "Generic connector, single row, 01x01, script generated (kicad-library-utils/schlib/autogen/connector/)"
 			(at 217.17 69.85 0)
 			(effects

Commit message: Fix Kicad
Parts:
- renumbered C26 to C24, C27 to C25, C28 to C26, J7 to J9, R18 to R16, R19 to R17, R20 to R18, R21 to R19, R22 to R20, R23 to R21, R24 to R22, R26 to R23, R25 to R24, R27 to R25, R28 to R26

Commit message: Update documentation
Parts:
- C24: symbol ESC-SchemSymLib:CL05B224KO5NNNC -> KururugiESC-Symbols-Lib:CL05B224KO5NNNC
- C25: symbol ESC-SchemSymLib:CL10A105KB8NNNC -> KururugiESC-Symbols-Lib:CL10A105KB8NNNC
- C26: symbol ESC-SchemSymLib:CL05B104KO5NNNC -> KururugiESC-Symbols-Lib:CL05B104KO5NNNC
- D5, D6, D7: symbol ESC-SchemSymLib:RB161QS-40T18R -> KururugiESC-Symbols-Lib:RB161QS-40T18R
- J9: symbol ESC-SchemSymLib:Conn_01x01_Phase -> KururugiESC-Symbols-Lib:Conn_01x01_Phase
- Q1, Q2: symbol ESC-SchemSymLib:CSD18540Q5B -> KururugiESC-Symbols-Lib:CSD18540Q5B
- R16, R18, R20: symbol ESC-SchemSymLib:0402WGJ033JTCE -> KururugiESC-Symbols-Lib:0402WGJ033JTCE
- R17, R21: symbol ESC-SchemSymLib:0402WGF100JTCE -> KururugiESC-Symbols-Lib:0402WGF100JTCE
- R19, R22, R23: symbol ESC-SchemSymLib:0402WGF1002TCE -> KururugiESC-Symbols-Lib:0402WGF1002TCE
- R24: symbol ESC-SchemSymLib:HoBB1216-5W-0.5mR-1% -> KururugiESC-Symbols-Lib:HoBB1216-5W-0.5mR-1%
- R25: symbol ESC-SchemSymLib:0402WGF330JTCE -> KururugiESC-Symbols-Lib:0402WGF330JTCE
- R26: symbol ESC-SchemSymLib:0402WGF1001TCE -> KururugiESC-Symbols-Lib:0402WGF1001TCE
- U4: symbol ESC-SchemSymLib:2EDL8024 -> KururugiESC-Symbols-Lib:2EDL8024
Changed lines of the file:
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@@
 	(text "PHASE"
 		(exclude_from_sim no)
-		(at 41.148 72.644 0)
+		(at 42.672 69.596 0)
 		(effects
 			(font
@@
 				(bold yes)
 			)
-			(justify left bottom)
+			(justify left top)
 		)
 	)
 	(text "BLDC PAD"
 		(exclude_from_sim no)
-		(at 182.245 56.515 0)
+		(at 182.626 52.832 0)
 		(effects
 			(font
@@
 				(bold yes)
 			)
-			(justify left bottom)
+			(justify left top)
 		)
 	)
 	(text "VOLTAGE SENSING"
 		(exclude_from_sim no)
-		(at 182.118 98.806 0)
+		(at 183.388 96.012 0)
 		(effects
 			(font
@@
 				(bold yes)
 			)
-			(justify left bottom)
+			(justify left top)
 		)
 	)
@@
 	)
 	(symbol
-		(lib_id "ESC-SchemSymLib:RB161QS-40T18R")
+		(lib_id "KururugiESC-Symbols-Lib:RB161QS-40T18R")
 		(at 85.09 81.28 180)
 		(unit 1)
@@
 	)
 	(symbol
-		(lib_id "ESC-SchemSymLib:0402WGF330JTCE")
+		(lib_id "KururugiESC-Symbols-Lib:0402WGF330JTCE")
 		(at 210.82 119.38 270)
 		(unit 1)
@@
 	)
 	(symbol
-		(lib_id "ESC-SchemSymLib:HoBB1216-5W-0.5mR-1%")
+		(lib_id "KururugiESC-Symbols-Lib:HoBB1216-5W-0.5mR-1%")
 		(at 148.59 115.57 0)
 		(unit 1)
@@
 	)
 	(symbol
-		(lib_id "ESC-SchemSymLib:0402WGJ033JTCE")
+		(lib_id "KururugiESC-Symbols-Lib:0402WGJ033JTCE")
 		(at 74.93 81.28 90)
 		(mirror x)
@@
 	)
 	(symbol
-		(lib_id "ESC-SchemSymLib:GND")
+		(lib_id "KururugiESC-Symbols-Lib:GND")
 		(at 52.07 99.06 0)
 		(unit 1)
@@
 	)
 	(symbol
-		(lib_id "ESC-SchemSymLib:0402WGJ033JTCE")
+		(lib_id "KururugiESC-Symbols-Lib:0402WGJ033JTCE")
 		(at 124.46 101.6 90)
 		(mirror x)
@@
 	)
 	(symbol
-		(lib_id "ESC-SchemSymLib:0402WGF1002TCE")
+		(lib_id "KururugiESC-Symbols-Lib:0402WGF1002TCE")
 		(at 133.35 111.76 0)
 		(unit 1)
@@
 	)
 	(symbol
-		(lib_id "ESC-SchemSymLib:GND")
+		(lib_id "KururugiESC-Symbols-Lib:GND")
 		(at 148.59 120.65 0)
 		(unit 1)
@@
 	)
 	(symbol
-		(lib_id "ESC-SchemSymLib:0402WGF1002TCE")
+		(lib_id "KururugiESC-Symbols-Lib:0402WGF1002TCE")
 		(at 133.35 90.17 0)
 		(unit 1)
@@
 	)
 	(symbol
-		(lib_id "ESC-SchemSymLib:GND")
+		(lib_id "KururugiESC-Symbols-Lib:GND")
 		(at 133.35 116.84 0)
 		(unit 1)
@@
 	)
 	(symbol
-		(lib_id "ESC-SchemSymLib:CL10A105KB8NNNC")
+		(lib_id "KururugiESC-Symbols-Lib:CL10A105KB8NNNC")
 		(at 52.07 92.71 0)
 		(mirror y)
@@
 	)
 	(symbol
-		(lib_id "ESC-SchemSymLib:GND")
+		(lib_id "KururugiESC-Symbols-Lib:GND")
 		(at 203.2 130.81 0)
 		(unit 1)
@@
 	)
 	(symbol
-		(lib_id "ESC-SchemSymLib:0402WGF1002TCE")
+		(lib_id "KururugiESC-Symbols-Lib:0402WGF1002TCE")
 		(at 203.2 113.03 0)
 		(unit 1)
@@
 	)
 	(symbol
-		(lib_id "ESC-SchemSymLib:Conn_01x01_Phase")
+		(lib_id "KururugiESC-Symbols-Lib:Conn_01x01_Phase")
 		(at 217.17 69.85 0)
 		(mirror x)
@@
 	)
 	(symbol
-		(lib_id "ESC-SchemSymLib:VDC")
+		(lib_id "KururugiESC-Symbols-Lib:VDC")
 		(at 52.07 86.36 0)
 		(mirror y)
@@
 	)
 	(symbol
-		(lib_id "ESC-SchemSymLib:RB161QS-40T18R")
+		(lib_id "KururugiESC-Symbols-Lib:RB161QS-40T18R")
 		(at 113.03 81.28 0)
 		(unit 1)
@@
 	)
 	(symbol
-		(lib_id "ESC-SchemSymLib:0402WGF1001TCE")
+		(lib_id "KururugiESC-Symbols-Lib:0402WGF1001TCE")
 		(at 203.2 125.73 180)
 		(unit 1)
@@
 	)
 	(symbol
-		(lib_id "ESC-SchemSymLib:CL05B224KO5NNNC")
+		(lib_id "KururugiESC-Symbols-Lib:CL05B224KO5NNNC")
 		(at 99.06 86.36 0)
 		(unit 1)
@@
 	)
 	(symbol
-		(lib_id "ESC-SchemSymLib:CL05B104KO5NNNC")
+		(lib_id "KururugiESC-Symbols-Lib:CL05B104KO5NNNC")
 		(at 218.44 125.73 0)
 		(unit 1)
@@
 	)
 	(symbol
-		(lib_id "ESC-SchemSymLib:0402WGJ033JTCE")
+		(lib_id "KururugiESC-Symbols-Lib:0402WGJ033JTCE")
 		(at 124.46 86.36 90)
 		(unit 1)
@@
 	)
 	(symbol
-		(lib_id "ESC-SchemSymLib:VDC")
+		(lib_id "KururugiESC-Symbols-Lib:VDC")
 		(at 148.59 78.74 0)
 		(mirror y)
@@
 	)
 	(symbol
-		(lib_id "ESC-SchemSymLib:2EDL8024")
+		(lib_id "KururugiESC-Symbols-Lib:2EDL8024")
 		(at 73.66 86.36 0)
 		(unit 1)
@@
 	)
 	(symbol
-		(lib_id "ESC-SchemSymLib:CSD18540Q5B")
+		(lib_id "KururugiESC-Symbols-Lib:CSD18540Q5B")
 		(at 146.05 86.36 0)
 		(unit 1)
@@
 	)
 	(symbol
-		(lib_id "ESC-SchemSymLib:RB161QS-40T18R")
+		(lib_id "KururugiESC-Symbols-Lib:RB161QS-40T18R")
 		(at 113.03 107.95 0)
 		(unit 1)
@@
 	)
 	(symbol
-		(lib_id "power:PWR_FLAG")
+		(lib_id "KururugiESC-Symbols-Lib:PWR_FLAG")
 		(at 208.28 69.85 0)
 		(unit 1)
@@
 	)
 	(symbol
-		(lib_id "ESC-SchemSymLib:GND")
+		(lib_id "KururugiESC-Symbols-Lib:GND")
 		(at 218.44 130.81 0)
 		(unit 1)
@@
 	)
 	(symbol
-		(lib_id "ESC-SchemSymLib:0402WGF100JTCE")
+		(lib_id "KururugiESC-Symbols-Lib:0402WGF100JTCE")
 		(at 124.46 81.28 90)
 		(unit 1)
@@
 	)
 	(symbol
-		(lib_id "ESC-SchemSymLib:0402WGF100JTCE")
+		(lib_id "KururugiESC-Symbols-Lib:0402WGF100JTCE")
 		(at 124.46 107.95 90)
 		(mirror x)
@@
 	)
 	(symbol
-		(lib_id "ESC-SchemSymLib:CSD18540Q5B")
+		(lib_id "KururugiESC-Symbols-Lib:CSD18540Q5B")
 		(at 146.05 101.6 0)
 		(unit 1)
